File: PCB/PCB.kicad_sch (KiCad schematic)
At the start: 10 parts, among them J1 Micro_SD_Card, U1 I2C, U2 DS3231MZ, U3 L7805

Commit message: PCB
Parts:
- removed U1: I2C, Package_TO_SOT_SMD:LFPAK56, symbol Analog_ADC:ADC101C021CIMK
- added C3: 0.33uF, Capacitor_THT:CP_Axial_L10.0mm_D4.5mm_P15.00mm_Horizontal, symbol Device:C
- added C4: 0.01uF, Capacitor_THT:CP_Axial_L10.0mm_D4.5mm_P15.00mm_Horizontal, symbol Device:C
- added Conn_FingerP1: Conn_FingerPrint, Connector_Molex:Molex_KK-254_AE-6410-04A_1x04_P2.54mm_Vertical, symbol PCM_4ms_Connector:Conn_01x04
- added Conn_Keypad1: Conn_Keypad, Connector_Molex:Molex_KK-254_AE-6410-08A_1x08_P2.54mm_Vertical, symbol PCM_4ms_Connector:Conn_01x08
- added Conn_RTC1: Conn_RTC, Connector_Molex:Molex_KK-254_AE-6410-06A_1x06_P2.54mm_Vertical, symbol PCM_4ms_Connector:Conn_01x06
- added Conn_SD1: Conn_SD, Connector_Molex:Molex_KK-254_AE-6410-08A_1x08_P2.54mm_Vertical, symbol PCM_4ms_Connector:Conn_01x08
- added J3: Conn_LCD, Connector_Molex:Molex_KK-254_AE-6410-04A_1x04_P2.54mm_Vertical, symbol PCM_4ms_Connector:Conn_01x04
- added L7805_1: L7805, Package_TO_SOT_THT:TO-220-3_Vertical, symbol Regulator_Linear:L7805
- added LED_B1: LCD battery, Battery:BatteryHolder_Eagle_12BH611-GR, symbol PCM_Elektuur:U
- added Sistem_B1: Sistem battery, Battery:BatteryHolder_Eagle_12BH611-GR, symbol PCM_Elektuur:U
- C1, C2: footprint Capacitor_THT:CP_Axial_L10.0mm_D6.0mm_P15.00mm_Horizontal -> Capacitor_THT:CP_Axial_L10.0mm_D4.5mm_P15.00mm_Horizontal
- U2: value DS3231MZ -> RTC
- renumbered BZ1 to Buzzer1, U3 to L7805_2
Connections:
- net GNDREF: now also A1.29 (GND), A2.7 (GND), Buzzer1.2 (+), C3.2, C4.1, Conn_FingerP1.1 (Pin_1), Conn_Keypad1.1 (Pin_1), Conn_RTC1.1 (Pin_1), Conn_SD1.8 (Pin_8), J3.1 (Pin_1), L7805_1.2 (GND), LED_B1.2 (-), Sistem_B1.2 (-); no longer J1.8 (GND), U2.1 (GND)
- net 5V+_Sistem: now reaches A2.8 (VIN)
- net 5V+_Sistem: now also A1.8 (VIN), Buzzer1.1 (-), C2.2, L7805_2.3 (OUT), Conn_Keypad1.2 (Pin_2), Conn_RTC1.2 (Pin_2), Conn_SD1.7 (Pin_7)
- removed net 5v+_componentes: C2.2, J1.6 (VSS), L7805_2.3 (OUT), U2.2 (VCC)
- net 9V+ renamed 9V+_Sistem
- net 9V+_Sistem: now also Sistem_B1.1 (+)
- new net 5V+_LCD: C4.2, Conn_FingerP1.2 (Pin_2), J3.2 (Pin_2), L7805_1.3 (OUT)
- new net 9V+_LCD: C3.1, L7805_1.1 (IN), LED_B1.1 (+)
Other:
- moved on the sheet: A1, A2, Buzzer1, C1, C2, DS1, J1, L7805_2, U2

Commit message: pcb
Parts:
- C1, C2, C3, C4: footprint Capacitor_THT:CP_Axial_L10.0mm_D4.5mm_P15.00mm_Horizontal -> Capacitor_SMD:C_0805_2012Metric_Pad1.18x1.45mm_HandSolder
Changed lines of the file:
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@@
+    )
+  )
+  (symbol (lib_id "Device:C") (at 75.565 34.925 90) (unit 1)
+    (in_bom yes) (on_board yes) (dnp no) (fields_autoplaced)
+    (property "Reference" "C4" (at 75.565 27.305 90)
+      (effects (font (size 1.27 1.27)))
+    )
+    (property "Value" "0.01uF" (at 75.565 29.845 90)
+      (effects (font (size 1.27 1.27)))
+    )
+    (property "Footprint" "Capacitor_SMD:C_0805_2012Metric_Pad1.18x1.45mm_HandSolder" (at 79.375 33.9598 0)
+      (effects (font (size 1.27 1.27)) hide)
+    )
+    (property "Datasheet" "~" (at 75.565 34.925 0)
+      (effects (font (size 1.27 1.27)) hide)
+    )
+    (pin "1")
+    (pin "2")
+    (instances
+      (project "PCB"
+        (path "/3c4caa8f-8861-413f-af61-fe2b5ea3fb26"
+          (reference "C4") (unit 1)
+        )
+      )
     )
   )
@@
       (effects (font (size 1.27 1.27)))
     )
-    (property "Footprint" "Capacitor_THT:CP_Axial_L10.0mm_D4.5mm_P15.00mm_Horizontal" (at 80.01 75.2348 0)
+    (property "Footprint" "Capacitor_SMD:C_0805_2012Metric_Pad1.18x1.45mm_HandSolder" (at 80.01 75.2348 0)
       (effects (font (size 1.27 1.27)) hide)
     )
@@
         (path "/3c4caa8f-8861-413f-af61-fe2b5ea3fb26"
           (reference "#PWR011") (unit 1)
-        )
-      )
-    )
-  )
-  (symbol (lib_id "Device:C") (at 56.515 28.575 0) (unit 1)
-    (in_bom yes) (on_board yes) (dnp no) (fields_autoplaced)
-    (property "Reference" "C3" (at 60.325 27.305 0)
-      (effects (font (size 1.27 1.27)) (justify left))
-    )
-    (property "Value" "0.33uF" (at 60.325 29.845 0)
-      (effects (font (size 1.27 1.27)) (justify left))
-    )
-    (property "Footprint" "Capacitor_THT:CP_Axial_L10.0mm_D4.5mm_P15.00mm_Horizontal" (at 57.4802 32.385 0)
-      (effects (font (size 1.27 1.27)) hide)
-    )
-    (property "Datasheet" "~" (at 56.515 28.575 0)
-      (effects (font (size 1.27 1.27)) hide)
-    )
-    (pin "1")
-    (pin "2")
-    (instances
-      (project "PCB"
-        (path "/3c4caa8f-8861-413f-af61-fe2b5ea3fb26"
-          (reference "C3") (unit 1)
         )
       )
@@
     )
   )
-  (symbol (lib_id "Device:C") (at 75.565 34.925 90) (unit 1)
-    (in_bom yes) (on_board yes) (dnp no) (fields_autoplaced)
-    (property "Reference" "C4" (at 75.565 27.305 90)
-      (effects (font (size 1.27 1.27)))
-    )
-    (property "Value" "0.01uF" (at 75.565 29.845 90)
-      (effects (font (size 1.27 1.27)))
-    )
-    (property "Footprint" "Capacitor_THT:CP_Axial_L10.0mm_D4.5mm_P15.00mm_Horizontal" (at 79.375 33.9598 0)
-      (effects (font (size 1.27 1.27)) hide)
-    )
-    (property "Datasheet" "~" (at 75.565 34.925 0)
-      (effects (font (size 1.27 1.27)) hide)
-    )
-    (pin "1")
-    (pin "2")
-    (instances
-      (project "PCB"
-        (path "/3c4caa8f-8861-413f-af61-fe2b5ea3fb26"
-          (reference "C4") (unit 1)
-        )
-      )
-    )
-  )
   (symbol (lib_id "Timer_RTC:DS3231MZ") (at 391.16 24.13 0) (unit 1)
     (in_bom yes) (on_board yes) (dnp no) (fields_autoplaced)
@@
         (path "/3c4caa8f-8861-413f-af61-fe2b5ea3fb26"
           (reference "#PWR09") (unit 1)
+        )
+      )
+    )
+  )
+  (symbol (lib_id "Device:C") (at 56.515 28.575 0) (unit 1)
+    (in_bom yes) (on_board yes) (dnp no) (fields_autoplaced)
+    (property "Reference" "C3" (at 60.325 27.305 0)
+      (effects (font (size 1.27 1.27)) (justify left))
+    )
+    (property "Value" "0.33uF" (at 60.325 29.845 0)
+      (effects (font (size 1.27 1.27)) (justify left))
+    )
+    (property "Footprint" "Capacitor_SMD:C_0805_2012Metric_Pad1.18x1.45mm_HandSolder" (at 57.4802 32.385 0)
+      (effects (font (size 1.27 1.27)) hide)
+    )
+    (property "Datasheet" "~" (at 56.515 28.575 0)
+      (effects (font (size 1.27 1.27)) hide)
+    )
+    (pin "1")
+    (pin "2")
+    (instances
+      (project "PCB"
+        (path "/3c4caa8f-8861-413f-af61-fe2b5ea3fb26"
+          (reference "C3") (unit 1)
         )
       )
@@
       (effects (font (size 1.27 1.27)) (justify left))
     )
-    (property "Footprint" "Capacitor_THT:CP_Axial_L10.0mm_D4.5mm_P15.00mm_Horizontal" (at 58.1152 73.66 0)
-      (effects (font (size 1.27 1.27)) hide)
-    )
+    (property "Footprint" "Capacitor_SMD:C_0805_2012Metric_Pad1.18x1.45mm_HandSolder" (at 58.1152 73.66 0)
+      (effects (font (size 1.27 1.27)) hide)
+    )

Commit message: envio PCB
Parts:
- removed Conn_SD1: Conn_SD, Connector_Molex:Molex_KK-254_AE-6410-08A_1x08_P2.54mm_Vertical, symbol PCM_4ms_Connector:Conn_01x08
- added Conn_SD1: Conn_RTC, Connector_Molex:Molex_KK-254_AE-6410-06A_1x06_P2.54mm_Vertical, symbol PCM_4ms_Connector:Conn_01x06
Connections:
- net 5V+_Sistem: now also Conn_SD1.5 (Pin_5); no longer Buzzer1.1 (-)
- net GNDREF: now also Conn_SD1.6 (Pin_6)
- net SCL_RTC: now reaches Conn_RTC1.3 (Pin_3)
- net SDA_RTC: now reaches Conn_RTC1.4 (Pin_4)
- net P2_keyPad: now reaches Conn_Keypad1.3 (Pin_3)
- net P3_keyPad: now reaches Conn_Keypad1.4 (Pin_4)
- net P4_keyPad: now reaches Conn_Keypad1.5 (Pin_5)
- net P5_keyPad: now reaches Conn_Keypad1.6 (Pin_6)
- net P6_keyPad: now reaches Conn_Keypad1.7 (Pin_7)
- net P7_keyPad: now reaches Conn_Keypad1.8 (Pin_8)
- net SDA_LCD: now reaches J3.3 (Pin_3)
- net SCL_LCD: now reaches J3.4 (Pin_4)
- new net CS: Conn_SD1.1 (Pin_1)
- new net MISO_SD: Conn_SD1.4 (Pin_4)
- new net MOSI_SD: Conn_SD1.3 (Pin_3)
- new net SCK: Conn_SD1.2 (Pin_2)
Other:
- moved on the sheet: Conn_Keypad1
