File: PCB/PCB.kicad_pcb (KiCad board)
At the start: 2 copper layers, 10 parts, among them J1 Micro_SD_Card, U1 I2C, U2 DS3231MZ, U3 L7805

Commit message: PCB
Parts:
- removed DS1: LCD 16X2, Display:WC1602A
- removed J1: Micro_SD_Card, Connector_Card:microSD_HC_Hirose_DM3AT-SF-PEJM5
- removed U1: I2C, Package_TO_SOT_SMD:LFPAK56
- removed U2: DS3231MZ, Package_SO:SO-16_3.9x9.9mm_P1.27mm
- added C3: 0.33uF, Capacitor_THT:CP_Axial_L10.0mm_D4.5mm_P15.00mm_Horizontal, F.Cu at (57.2, 105.1)
- added C4: 0.01uF, Capacitor_THT:CP_Axial_L10.0mm_D4.5mm_P15.00mm_Horizontal, F.Cu at (65.7, 120.1)
- added Conn_FingerP1: Conn_FingerPrint, Connector_Molex:Molex_KK-254_AE-6410-04A_1x04_P2.54mm_Vertical, F.Cu at (65.8, 133.5)
- added Conn_Keypad1: Conn_Keypad, Connector_Molex:Molex_KK-254_AE-6410-08A_1x08_P2.54mm_Vertical, F.Cu at (77.5, 137.0)
- added Conn_RTC1: Conn_RTC, Connector_Molex:Molex_KK-254_AE-6410-06A_1x06_P2.54mm_Vertical, F.Cu at (80.2, 127.5)
- added Conn_SD1: Conn_SD, Connector_Molex:Molex_KK-254_AE-6410-08A_1x08_P2.54mm_Vertical, F.Cu at (77.3, 146.2)
- added J3: Conn_LCD, Connector_Molex:Molex_KK-254_AE-6410-04A_1x04_P2.54mm_Vertical, F.Cu at (56.8, 133.6)
- added L7805_1: L7805, Package_TO_SOT_THT:TO-220-3_Vertical, F.Cu at (59.2, 98.6)
- added LED_B1: LCD battery, Battery:BatteryHolder_Eagle_12BH611-GR, F.Cu at (41.2, 98.6)
- added Sistem_B1: Sistem battery, Battery:BatteryHolder_Eagle_12BH611-GR, F.Cu at (121.5, 98.3)
- A1, A2: moved to B.Cu
- C1, C2: footprint Capacitor_THT:CP_Axial_L10.0mm_D6.0mm_P15.00mm_Horizontal -> Capacitor_THT:CP_Axial_L10.0mm_D4.5mm_P15.00mm_Horizontal
- moved A1 177.8 mm to (21.9, 50.6), turned to -90 degrees
- moved C2 141.6 mm to (78.2, 119.8)
- moved Buzzer1 135.0 mm to (57.2, 144.8)
- moved C1 118.5 mm to (88.3, 104.8), turned to -90 degrees
- moved L7805_2 112.1 mm to (86.5, 97.0), turned to 180 degrees
- moved A2 97.7 mm to (79.2, 50.1), turned to -90 degrees
- renumbered BZ1 to Buzzer1, U3 to L7805_2
Connections:
- net 9V+ renamed 9V+_Sistem
- A1 pad 13: Net-(A1-SDA/A4) -> unconnected-(A1-SDA/A4-Pad13)
- A1 pad 14: Net-(A1-SCL/A5) -> unconnected-(A1-SCL/A5-Pad14)
- A1 pad 15: Net-(A1-D0/RX) -> unconnected-(A1-D0/RX-Pad15)
- A1 pad 16: Net-(A1-D1/TX) -> unconnected-(A1-D1/TX-Pad16)
- A1 pad 2: (no net) -> unconnected-(A1-IOREF-Pad2)
- A1 pad 29: (no net) -> GNDREF
- A1 pad 30: (no net) -> unconnected-(A1-AREF-Pad30)
- A1 pad 8: (no net) -> 5V+_Sistem
- A2 pad 15: Net-(A1-D0/RX) -> unconnected-(A2-D0/RX-Pad15)
- A2 pad 16: Net-(A1-D1/TX) -> unconnected-(A2-D1/TX-Pad16)
- A2 pad 2: (no net) -> unconnected-(A2-IOREF-Pad2)
- A2 pad 29: (no net) -> unconnected-(A2-GND-Pad29)
- A2 pad 30: (no net) -> unconnected-(A2-AREF-Pad30)
- A2 pad 7: unconnected-(A2-GND-Pad7) -> GNDREF
- A2 pad 8: (no net) -> 5V+_Sistem
- Buzzer1 pad 1: unconnected-(BZ1---Pad1) -> 5V+_Sistem
- Buzzer1 pad 2: unconnected-(BZ1-+-Pad2) -> GNDREF
- C2 pad 2: 5v+_componentes -> 5V+_Sistem
- L7805_2 pad 3: 5v+_componentes -> 5V+_Sistem
Routing:
- net 5V+_Sistem: track 0.00 -> 182.8 mm
- net 5V+_LCD: track 0.00 -> 48.6 mm
- net 9V+_Sistem: track 0.00 -> 46.7 mm
- net 9V+_LCD: track 0.00 -> 25.3 mm
- added copper zone on F.Cu, net GNDREF
Other:
- board text added: "A_Master"
- board text added: "A_Slave"
- board text added: "Conn_LCD"

Commit message: pcb
Parts:
- C1, C2, C3, C4: footprint Capacitor_THT:CP_Axial_L10.0mm_D4.5mm_P15.00mm_Horizontal -> Capacitor_SMD:C_0805_2012Metric_Pad1.18x1.45mm_HandSolder
- moved C4 52.4 mm to (39.5, 165.5), turned to 0 degrees
- moved C3 11.3 mm to (66.2, 111.8), turned to 90 degrees
Connections:
- C3 pad 1: 9V+_LCD -> (no net)
- C3 pad 2: GNDREF -> (no net)
Other:
- board text added: "RTC"

Commit message: PCB
Parts:
- removed Conn_FingerP1: Conn_FingerPrint, Connector_Molex:Molex_KK-254_AE-6410-04A_1x04_P2.54mm_Vertical
- moved C4 66.2 mm to (64.3, 104.1), turned to 90 degrees
- moved J3 17.8 mm to (58.7, 115.8), turned to 0 degrees
- moved C2 16.0 mm to (81.5, 104.1)
- moved Conn_RTC1 11.8 mm to (78.5, 115.8)
- moved C3 10.4 mm to (59.2, 104.1), turned to -90 degrees
- moved Buzzer1 10.2 mm to (58.4, 134.6)
- moved Conn_Keypad1 8.85 mm to (75.9, 128.3)
- moved Conn_SD1 5.53 mm to (75.7, 141.0)
- moved Sistem_B1 3.55 mm to (119.0, 95.8)
- moved LED_B1 2.20 mm to (41.9, 96.5)
- moved C1 1.75 mm to (86.6, 104.1)
Connections:
- C3 pad 1: (no net) -> 9V+_LCD
- C3 pad 2: (no net) -> GNDREF
Routing:
- net 5V+_Sistem: track 182.8 -> 88.7 mm
- net 5V+_LCD: track 48.6 -> 0.00 mm
- net 9V+_Sistem: track 46.7 -> 0.04 mm
- net 9V+_LCD: track 25.3 -> 0.01 mm
Other:
- board text removed: "RTC"

Commit message: envio PCB
Parts:
- added A1: Master, Module:Arduino_UNO_R3, B.Cu at (143.7, 53.2)
- added A2: Slave, Module:Arduino_UNO_R3, B.Cu at (201.1, 52.8)
- added Buzzer1: Buzzer, Buzzer_Beeper:MagneticBuzzer_ProSignal_ABI-010-RC, F.Cu at (203.5, 138.9)
- added C1: 0.33uF, Capacitor_SMD:C_0805_2012Metric_Pad1.18x1.45mm_HandSolder, F.Cu at (208.4, 106.8)
- added C2: 0.01uF, Capacitor_SMD:C_0805_2012Metric_Pad1.18x1.45mm_HandSolder, F.Cu at (203.4, 106.8)
- added C3: 0.33uF, Capacitor_SMD:C_0805_2012Metric_Pad1.18x1.45mm_HandSolder, F.Cu at (181.0, 106.8)
- added C4: 0.01uF, Capacitor_SMD:C_0805_2012Metric_Pad1.18x1.45mm_HandSolder, F.Cu at (186.1, 106.8)
- added Conn_Keypad1: Conn_Keypad, Connector_Molex:Molex_KK-254_AE-6410-08A_1x08_P2.54mm_Vertical, F.Cu at (179.3, 144.0)
- added Conn_RTC1: Conn_RTC, Connector_Molex:Molex_KK-254_AE-6410-06A_1x06_P2.54mm_Vertical, F.Cu at (200.3, 118.5)
- added Conn_SD1: Conn_SD, Connector_Molex:Molex_KK-254_AE-6410-08A_1x08_P2.54mm_Vertical, F.Cu at (191.6, 126.3)
- added J3: Conn_LCD, Connector_Molex:Molex_KK-254_AE-6410-04A_1x04_P2.54mm_Vertical, F.Cu at (184.8, 120.5)
- added L7805_1: L7805, Package_TO_SOT_THT:TO-220-3_Vertical, F.Cu at (181.0, 101.2)
- added L7805_2: L7805, Package_TO_SOT_THT:TO-220-3_Vertical, F.Cu at (208.4, 99.6)
- added LED_B1: LCD battery, Battery:BatteryHolder_Eagle_12BH611-GR, F.Cu at (163.7, 99.2)
- added Sistem_B1: Sistem battery, Battery:BatteryHolder_Eagle_12BH611-GR, F.Cu at (240.9, 98.4)
- moved Sistem_B1 49.8 mm to (107.8, 144.2), turned to -90 degrees
- moved Buzzer1 23.3 mm to (81.7, 136.2)
- moved Conn_Keypad1 22.6 mm to (57.5, 141.4), turned to 90 degrees
- moved Conn_SD1 18.3 mm to (69.8, 123.7), turned to -90 degrees
- moved J3 4.76 mm to (63.0, 117.8), turned to 90 degrees
Connections:
- A1 pad 31: unconnected-(A1-SDA/A4-Pad31) -> SDA_LCD
- A1 pad 32: unconnected-(A1-SCL/A5-Pad32) -> SCL_LCD
- Buzzer1 pad 1: 5V+_Sistem -> unconnected-(Buzzer1---Pad1)
- Conn_Keypad1 pad 3: unconnected-(Conn_Keypad1-Pin_3-Pad3) -> P2_keyPad
- Conn_Keypad1 pad 4: unconnected-(Conn_Keypad1-Pin_4-Pad4) -> P3_keyPad
- Conn_Keypad1 pad 5: unconnected-(Conn_Keypad1-Pin_5-Pad5) -> P4_keyPad
- Conn_Keypad1 pad 6: unconnected-(Conn_Keypad1-Pin_6-Pad6) -> P5_keyPad
- Conn_Keypad1 pad 7: unconnected-(Conn_Keypad1-Pin_7-Pad7) -> P6_keyPad
- Conn_Keypad1 pad 8: unconnected-(Conn_Keypad1-Pin_8-Pad8) -> P7_keyPad
- Conn_RTC1 pad 3: unconnected-(Conn_RTC1-Pin_3-Pad3) -> SCL_RTC
- Conn_RTC1 pad 4: unconnected-(Conn_RTC1-Pin_4-Pad4) -> SDA_RTC
- J3 pad 3: unconnected-(J3-Pin_3-Pad3) -> SDA_LCD
- J3 pad 4: unconnected-(J3-Pin_4-Pad4) -> SCL_LCD
Routing:
- net 5V+_Sistem: track 88.7 -> 425.4 mm
- net SCL_LCD: track 0.00 -> 160.3 mm
- net SDA_LCD: track 0.00 -> 158.7 mm
- net unconnected-(A2-SCL/A5-Pad32): track 0.00 -> 148.9 mm
- net unconnected-(A2-SDA/A4-Pad31): track 0.00 -> 141.8 mm
- net unconnected-(Buzzer1---Pad1): track 0.00 -> 100.7 mm, vias 0 -> 4
- net 9V+_Sistem: track 0.04 -> 87.8 mm
- net unconnected-(A2-D4-Pad19): track 0.00 -> 78.8 mm
- net SCL_RTC: track 0.00 -> 55.0 mm, vias 0 -> 4
- net SDA_RTC: track 0.00 -> 52.3 mm, vias 0 -> 4
- net 5V+_LCD: track 0.00 -> 45.3 mm
- net 9V+_LCD: track 0.01 -> 45.3 mm

Commit message: trilhas PCB
Parts:
- removed the A1 at (143.7, 53.2)
- removed the A2 at (201.1, 52.8)
- removed the Buzzer1 at (203.5, 138.9)
- removed the C1 at (208.4, 106.8)
- removed the C2 at (203.4, 106.8)
- removed the C3 at (181.0, 106.8)
- removed the C4 at (186.1, 106.8)
- removed the Conn_Keypad1 at (179.3, 144.0)
- removed the Conn_RTC1 at (200.3, 118.5)
- removed the Conn_SD1 at (69.8, 123.7)
- removed the Conn_SD1 at (191.6, 126.3)
- removed the J3 at (184.8, 120.5)
- removed the L7805_1 at (181.0, 101.2)
- removed the L7805_2 at (208.4, 99.6)
- removed the LED_B1 at (163.7, 99.2)
- removed the Sistem_B1 at (240.9, 98.4)
- added Conn_SD1: Conn_RTC, Connector_Molex:Molex_KK-254_AE-6410-06A_1x06_P2.54mm_Vertical, F.Cu at (89.7, 110.7)
- moved C1 40.7 mm to (87.7, 144.9)
- moved C2 40.7 mm to (82.6, 144.9)
- moved L7805_2 40.7 mm to (87.6, 137.7)
- moved Buzzer1 18.6 mm to (94.7, 122.9), turned to 180 degrees
- moved Conn_RTC1 18.2 mm to (76.6, 97.7), turned to -90 degrees
- moved J3 6.18 mm to (57.1, 115.8)
- moved C3 4.22 mm to (55.6, 101.9)
- moved C4 4.22 mm to (60.7, 101.9)
- moved L7805_1 4.22 mm to (55.6, 96.3)
- moved Sistem_B1 0.99 mm to (108.8, 144.2)
Connections:
- A1 pad 13: unconnected-(A1-SDA/A4-Pad13) -> SDA_MS
- A1 pad 14: unconnected-(A1-SCL/A5-Pad14) -> SCL_MS
- A1 pad 17: unconnected-(A1-D2-Pad17) -> P2_keyPad
- A1 pad 18: unconnected-(A1-D3-Pad18) -> P3_keyPad
- A1 pad 19: unconnected-(A1-D4-Pad19) -> P4_keyPad
- A1 pad 20: unconnected-(A1-D5-Pad20) -> P5_keyPad
- A1 pad 21: unconnected-(A1-D6-Pad21) -> P6_keyPad
- A1 pad 22: unconnected-(A1-D7-Pad22) -> P7_keyPad
- A1 pad 23: unconnected-(A1-D8-Pad23) -> (no net)
- A2 pad 13: unconnected-(A2-SDA/A4-Pad13) -> SDA_MS
- A2 pad 14: unconnected-(A2-SCL/A5-Pad14) -> SCL_MS
- A2 pad 19: unconnected-(A2-D4-Pad19) -> unconnected-(Buzzer1---Pad1)
- A2 pad 25: unconnected-(A2-D10-Pad25) -> CS
- A2 pad 26: unconnected-(A2-D11-Pad26) -> MOSI_SD
- A2 pad 27: unconnected-(A2-D12-Pad27) -> MISO_SD
- A2 pad 28: unconnected-(A2-D13-Pad28) -> SCK
- A2 pad 31: unconnected-(A2-SDA/A4-Pad31) -> SDA_RTC
- A2 pad 32: unconnected-(A2-SCL/A5-Pad32) -> SCL_RTC
Routing:
- net 5V+_Sistem: track 425.4 -> 154.9 mm, vias 0 -> 2
- net unconnected-(A2-SCL/A5-Pad32): track 148.9 -> 0.00 mm
- net unconnected-(A2-SDA/A4-Pad31): track 141.8 -> 0.00 mm
- net SCL_LCD: track 160.3 -> 77.4 mm
- net SDA_LCD: track 158.7 -> 77.8 mm
- net SCK: track 0.00 -> 79.7 mm
- net unconnected-(A2-D4-Pad19): track 78.8 -> 0.00 mm
- net P7_keyPad: track 0.00 -> 71.9 mm
- net CS: track 0.00 -> 70.9 mm
- net P6_keyPad: track 0.00 -> 70.0 mm
- net MISO_SD: track 0.00 -> 68.4 mm
- net P5_keyPad: track 0.00 -> 68.1 mm
- net P2_keyPad: track 0.00 -> 67.9 mm
- net MOSI_SD: track 0.00 -> 67.4 mm
- net P4_keyPad: track 0.00 -> 66.8 mm
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